Commit message: Imported upstream version '0.9.4' of 'upstream'

File: diff_drive_controller/test/sphere_wheel.xacro (robot description, xacro)
@@ -1,5 +1,5 @@
 <?xml version="1.0"?>
 <robot xmlns:xacro="http://www.ros.org/wiki/xacro">
-  <xacro:macro name="sphere_wheel" params="name parent radius *origin">
+  <macro name="sphere_wheel" params="name parent radius *origin">
     <link name="${name}_link">
       <inertial>
@@ -24,5 +24,5 @@
       <parent link="${parent}_link"/>
       <child link="${name}_link"/>
-      <xacro:insert_block name="origin"/>
+      <insert_block name="origin"/>
       <axis xyz="0 0 1"/>
     </joint>
@@ -37,4 +37,4 @@
       <material>Gazebo/Red</material>
     </gazebo>
-  </xacro:macro>
+  </macro>
 </robot>

File: diff_drive_controller/test/wheel.xacro (robot description, xacro)
@@ -1,5 +1,5 @@
 <?xml version="1.0"?>
 <robot xmlns:xacro="http://www.ros.org/wiki/xacro">
-  <xacro:macro name="wheel" params="name parent radius thickness *origin">
+  <macro name="wheel" params="name parent radius thickness *origin">
     <link name="${name}_link">
       <inertial>
@@ -24,5 +24,5 @@
       <parent link="${parent}_link"/>
       <child link="${name}_link"/>
-      <xacro:insert_block name="origin"/>
+      <insert_block name="origin"/>
       <axis xyz="0 0 1"/>
     </joint>
@@ -37,4 +37,4 @@
       <material>Gazebo/Red</material>
     </gazebo>
-  </xacro:macro>
+  </macro>
 </robot>
