Commit message: Imported upstream version '0.13.0' of 'upstream'

File: diff_drive_controller/test/square_wheel.xacro (robot description, xacro)
@@ -1,5 +1,5 @@
 <?xml version="1.0"?>
 <robot xmlns:xacro="http://www.ros.org/wiki/xacro">
-  <xacro:macro name="wheel" params="name parent radius thickness *origin">
+  <macro name="square_wheel" params="name parent radius *origin">
     <link name="${name}_link">
       <inertial>
@@ -11,5 +11,6 @@
         <origin xyz="0 0 0" rpy="0 0 0"/>
         <geometry>
-          <cylinder radius="${wheel_radius}" length="${thickness}"/>
+          <!-- use boxes for wheels, scale radius to account for "circumference" difference -->
+          <box size="${wheel_radius*1.11} ${wheel_radius*1.11} ${wheel_radius*1.11} "/>
         </geometry>
       </visual>
@@ -17,5 +18,5 @@
         <origin xyz="0 0 0" rpy="0 0 0"/>
         <geometry>
-          <cylinder radius="${wheel_radius}" length="${thickness}"/>
+          <box size="${wheel_radius*1.11} ${wheel_radius*1.11} ${wheel_radius*1.11} "/>
         </geometry>
       </collision>
@@ -24,5 +25,5 @@
       <parent link="${parent}_link"/>
       <child link="${name}_link"/>
-      <xacro:insert_block name="origin"/>
+      <insert_block name="origin"/>
       <axis xyz="0 0 1"/>
     </joint>
@@ -37,4 +38,4 @@
       <material>Gazebo/Red</material>
     </gazebo>
-  </xacro:macro>
+  </macro>
 </robot>

Commit message: Imported upstream version '0.14.0' of 'upstream'

File: diff_drive_controller/test/square_wheel.xacro (robot description, xacro)
@@ -1,5 +1,5 @@
 <?xml version="1.0"?>
 <robot xmlns:xacro="http://www.ros.org/wiki/xacro">
-  <macro name="square_wheel" params="name parent radius *origin">
+  <xacro:macro name="square_wheel" params="name parent radius *origin">
     <link name="${name}_link">
       <inertial>
@@ -25,5 +25,5 @@
       <parent link="${parent}_link"/>
       <child link="${name}_link"/>
-      <insert_block name="origin"/>
+      <xacro:insert_block name="origin"/>
       <axis xyz="0 0 1"/>
     </joint>
@@ -38,4 +38,4 @@
       <material>Gazebo/Red</material>
     </gazebo>
-  </macro>
+  </xacro:macro>
 </robot>
