Commit message: Rebase from 'upstream'

File: effort_controllers/test/simple_bot.xacro (robot description, xacro)
@@ -16,13 +16,3 @@
     <limit lower="-6.3" upper="6.3" effort="10" velocity="2"/>
   </joint>
-  <transmission name="transimssion">
-    <type>transmission_interface/SimpleTransmission</type>
-    <joint name="joint">
-      <hardwareInterface>hardware_interface/EffortJointInterface</hardwareInterface>
-    </joint>
-    <actuator name="motor">
-      <hardwareInterface>hardware_interface/EffortJointInterface</hardwareInterface>
-      <mechanicalReduction>1</mechanicalReduction>
-    </actuator>
-  </transmission>
 </robot>

Commit message: Imported upstream version '0.17.3' of 'upstream'

File: effort_controllers/test/simple_bot.xacro (robot description, xacro)
@@ -16,3 +16,13 @@
     <limit lower="-6.3" upper="6.3" effort="10" velocity="2"/>
   </joint>
+  <transmission name="transimssion">
+    <type>transmission_interface/SimpleTransmission</type>
+    <joint name="joint">
+      <hardwareInterface>hardware_interface/EffortJointInterface</hardwareInterface>
+    </joint>
+    <actuator name="motor">
+      <hardwareInterface>hardware_interface/EffortJointInterface</hardwareInterface>
+      <mechanicalReduction>1</mechanicalReduction>
+    </actuator>
+  </transmission>
 </robot>
